File: rv_9_schematic_3.sch (KiCad schematic (older format))
At the start: 7 parts, among them M1 Flap Motor, SW5 SW_DPDT_on-off-on, SW6 SW_SPST

Commit message: new version kicad changes
Parts:
- B3: symbol BUS-BAR -> AvionicSchematic:BUS-BAR
- F7: symbol Fuse -> rv_9_schematic-rescue:Fuse
- G15, G16: symbol LCL -> AvionicSchematic:LCL
- M1: symbol Motor_DC -> AvionicSchematic:Motor_DC
- SW5: symbol SW_DPDT_on-off-on -> AvionicSchematic:SW_DPDT_on-off-on
- SW6: symbol SW_SPST -> rv_9_schematic-rescue:SW_SPST
Changed lines of the file:
@@
-EESchema Schematic File Version 2
-LIBS:power
-LIBS:device
-LIBS:switches
-LIBS:relays
-LIBS:motors
-LIBS:transistors
-LIBS:conn
-LIBS:linear
-LIBS:regul
-LIBS:74xx
-LIBS:cmos4000
-LIBS:adc-dac
-LIBS:memory
-LIBS:xilinx
-LIBS:microcontrollers
-LIBS:dsp
-LIBS:microchip
-LIBS:analog_switches
-LIBS:motorola
-LIBS:texas
-LIBS:intel
-LIBS:audio
-LIBS:interface
-LIBS:digital-audio
-LIBS:philips
-LIBS:display
-LIBS:cypress
-LIBS:siliconi
-LIBS:opto
-LIBS:atmel
-LIBS:contrib
-LIBS:valves
-LIBS:AvionicSchematic
-LIBS:rv_9_schematic-cache
-EELAYER 25 0
+EESchema Schematic File Version 4
+EELAYER 30 0
 EELAYER END
 $Descr USLetter 11000 8500
@@
 $EndDescr
 $Comp
-L BUS-BAR B3
+L AvionicSchematic:BUS-BAR B3
 U 1 1 5B79C072
 P 2575 6525
@@
 $EndComp
 $Comp
-L Fuse F7
+L rv_9_schematic-rescue:Fuse F7
 U 1 1 5B79C1B1
 P 2900 6200
+AR Path="/5B79C1B1" Ref="F7"  Part="1"
+AR Path="/5B79C069/5B79C1B1" Ref="F7"  Part="1"
 F 0 "F7" V 2980 6200 50  0000 C CNN
 F 1 "Fuse" V 2825 6200 50  0000 C CNN
@@
 $EndComp
 $Comp
-L SW_SPST SW6
+L rv_9_schematic-rescue:SW_SPST SW6
 U 1 1 5B79C317
 P 5150 3950
@@
 $EndComp
 $Comp
-L Motor_DC M1
+L AvionicSchematic:Motor_DC M1
 U 1 1 5B79C3CE
 P 5400 4975
@@
 $EndComp
 $Comp
-L SW_DPDT_on-off-on SW5
+L AvionicSchematic:SW_DPDT_on-off-on SW5
 U 1 1 5B79CFC7
 P 3825 5000
@@
 	4025 4700 4150 4700
 $Comp
-L LCL G15
+L AvionicSchematic:LCL G15
 U 1 1 5B79D46D
 P 3250 5600
@@
 	3250 5150 3250 5325
 $Comp
-L LCL G16
+L AvionicSchematic:LCL G16
 U 1 1 5B79D675
 P 5475 4325
