File: rv_9_schematic_4.sch (KiCad schematic (older format))
At the start: 5 parts, among them SW7 SW_SPST

Commit message: new version kicad changes
Parts:
- B4: symbol BUS-BAR -> AvionicSchematic:BUS-BAR
- F8: symbol Fuse -> rv_9_schematic-rescue:Fuse
- G17: symbol LCL -> AvionicSchematic:LCL
- SW7: symbol SW_SPST -> rv_9_schematic-rescue:SW_SPST
- U?: symbol NavCom -> AvionicSchematic:NavCom
Changed lines of the file:
@@
-EESchema Schematic File Version 2
-LIBS:power
-LIBS:device
-LIBS:switches
-LIBS:relays
-LIBS:motors
-LIBS:transistors
-LIBS:conn
-LIBS:linear
-LIBS:regul
-LIBS:74xx
-LIBS:cmos4000
-LIBS:adc-dac
-LIBS:memory
-LIBS:xilinx
-LIBS:microcontrollers
-LIBS:dsp
-LIBS:microchip
-LIBS:analog_switches
-LIBS:motorola
-LIBS:texas
-LIBS:intel
-LIBS:audio
-LIBS:interface
-LIBS:digital-audio
-LIBS:philips
-LIBS:display
-LIBS:cypress
-LIBS:siliconi
-LIBS:opto
-LIBS:atmel
-LIBS:contrib
-LIBS:valves
-LIBS:AvionicSchematic
-LIBS:rv_9_schematic-cache
-EELAYER 25 0
+EESchema Schematic File Version 4
+EELAYER 30 0
 EELAYER END
 $Descr A 11000 8500
@@
 $EndDescr
 $Comp
-L BUS-BAR B4
+L AvionicSchematic:BUS-BAR B4
 U 1 1 5B7AF662
 P 2325 6275
@@
 $EndComp
 $Comp
-L LCL G17
+L AvionicSchematic:LCL G17
 U 1 1 5B7AF759
 P 4175 6875
@@
 $EndComp
 $Comp
-L SW_SPST SW7
+L rv_9_schematic-rescue:SW_SPST SW7
 U 1 1 5B7AF820
 P 3775 5400
@@
 $EndComp
 $Comp
-L Fuse F8
+L rv_9_schematic-rescue:Fuse F8
 U 1 1 5B7AF8D1
 P 2375 5375
+AR Path="/5B7AF8D1" Ref="F8"  Part="1"
+AR Path="/5B7AF59F/5B7AF8D1" Ref="F8"  Part="1"
 F 0 "F8" V 2455 5375 50  0000 C CNN
 F 1 "Fuse" V 2300 5375 50  0000 C CNN
@@
 E-BUS
 $Comp
-L NavCom U?
+L AvionicSchematic:NavCom U?
 U 1 1 5B7B770E
 P 6250 5300
