File: rv_9_schematic_5.sch (KiCad schematic (older format))
At the start: 5 parts

Commit message: new version kicad changes
Parts:
- B? (x2): symbol BUS-BAR -> AvionicSchematic:BUS-BAR
- F?: symbol Fuse -> rv_9_schematic-rescue:Fuse
- K?: symbol G5Q-1 -> rv_9_schematic-rescue:G5Q-1
- SW?: symbol SW_SPDT -> rv_9_schematic-rescue:SW_SPDT
Changed lines of the file:
@@
-EESchema Schematic File Version 2
-LIBS:power
-LIBS:device
-LIBS:switches
-LIBS:relays
-LIBS:motors
-LIBS:transistors
-LIBS:conn
-LIBS:linear
-LIBS:regul
-LIBS:74xx
-LIBS:cmos4000
-LIBS:adc-dac
-LIBS:memory
-LIBS:xilinx
-LIBS:microcontrollers
-LIBS:dsp
-LIBS:microchip
-LIBS:analog_switches
-LIBS:motorola
-LIBS:texas
-LIBS:intel
-LIBS:audio
-LIBS:interface
-LIBS:digital-audio
-LIBS:philips
-LIBS:display
-LIBS:cypress
-LIBS:siliconi
-LIBS:opto
-LIBS:atmel
-LIBS:contrib
-LIBS:valves
-LIBS:AvionicSchematic
-LIBS:rv_9_schematic-cache
-EELAYER 25 0
+EESchema Schematic File Version 4
+EELAYER 30 0
 EELAYER END
 $Descr A4 11693 8268
@@
 $EndDescr
 $Comp
-L BUS-BAR B?
+L AvionicSchematic:BUS-BAR B?
 U 1 1 5B7B8663
 P 2000 3000
@@
 $EndComp
 $Comp
-L BUS-BAR B?
+L AvionicSchematic:BUS-BAR B?
 U 1 1 5B7B87DA
 P 1950 3675
@@
 $EndComp
 $Comp
-L Fuse F?
+L rv_9_schematic-rescue:Fuse F?
 U 1 1 5B7B886B
 P 3575 4425
+AR Path="/5B7B886B" Ref="F?"  Part="1"
+AR Path="/5B7B854A/5B7B886B" Ref="F?"  Part="1"
 F 0 "F?" V 3655 4425 50  0000 C CNN
 F 1 "Fuse" V 3500 4425 50  0000 C CNN
@@
 $EndComp
 $Comp
-L G5Q-1 K?
+L rv_9_schematic-rescue:G5Q-1 K?
 U 1 1 5B7B891E
 P 3450 2200
@@
 $EndComp
 $Comp
-L SW_SPDT SW?
+L rv_9_schematic-rescue:SW_SPDT SW?
 U 1 1 5B7B89DF
 P 3900 3375
